Commit message: add ur5 namespace

File: arm_gazebo/urdf/ur_gripper.urdf.xacro (robot description, xacro)
@@ -6,5 +6,5 @@
   <xacro:include filename="$(find robotiq_ft_sensor)/urdf/robotiq_ft300.urdf.xacro" />
   <xacro:include filename="$(find robotiq_85_description)/urdf/robotiq_85_gripper.urdf.xacro" />
-  <xacro:ur5_robot prefix="" joint_limited="false"
+  <xacro:ur5_robot prefix="ur5/" joint_limited="false"
     transmission_hw_interface="$(arg transmission_hw_interface)"
   />
@@ -12,8 +12,8 @@
   <joint name="world_joint" type="fixed">
     <parent link="world" />
-    <child link = "base_link" />
+    <child link = "ur5/base_link" />
     <origin xyz="0.0 0.0 0.0" rpy="0.0 0.0 0.0" />
   </joint>
-  <xacro:robotiq_ft300 prefix="" parent="tool0" >
+  <xacro:robotiq_ft300 prefix="" parent="ur5/tool0" >
 		<origin xyz="0 0 0" rpy="0 0 ${-pi/2}"/>
 	</xacro:robotiq_ft300>

File: robotiq_85_description/urdf/robotiq_85_gripper.urdf.xacro (robot description, xacro)
@@ -303,5 +303,5 @@
             <arm>
               <arm_name>gripper_arm</arm_name>
-              <palm_link>wrist_3_link</palm_link>
+              <palm_link>ur5/wrist_3_link</palm_link>
               <gripper_link>${prefix}gripper_finger1_finger_tip_link</gripper_link>
               <gripper_link>${prefix}gripper_finger2_finger_tip_link</gripper_link>
