Commit message: gripper bumper

File: robotiq_85_description/urdf/robotiq_85_gripper.urdf.xacro (robot description, xacro)
@@ -292,4 +292,46 @@
             </inertial>
         </link>
+        <!-- #############################bumper_test###############################-->
+        <link name="${prefix}bumper_gripper_link">
+          <inertial>
+              <origin rpy="0 0 0" xyz="0 0 0"/>
+              <mass value="0.0000000000001"/>
+              <inertia ixx="0.00000001" ixy="0.00000001" ixz="0.00000001" iyy="0.00000001" iyz="0.00000001" izz="0.00000001"/>
+          </inertial>
+          <!-- <visual>
+              <origin rpy="0 0 0" xyz="0.168 0 0"/>
+              <geometry>
+                  <box size="0.01 0.13 0.11"/>
+              </geometry>
+              <material name="red">
+                  <color rgba="1.0 0.0 0.0 1.0"/>
+              </material>
+          </visual> -->
+          <collision name="${prefix}gripper_base_link_fixed_joint_lump__${prefix}/bumper_gripper_link">
+              <origin rpy="0 0 0" xyz="0.168 0 0"/>
+              <geometry>
+                  <box size="0.01 0.13 0.11"/>
+              </geometry>
+          </collision>
+        </link>
+        <joint name="${prefix}bumper_gripper_joint" type="fixed">
+            <origin xyz="0 0 0" rpy="0.0 0.0 0.0"/>
+            <parent link="${prefix}gripper_base_link" />
+            <child link="${prefix}bumper_gripper_link" />
+        </joint>
+        <gazebo reference="${prefix}bumper_gripper_link">
+          <sensor name='contactsensor_sensor' type='contact'>
+            <always_on>true</always_on>
+            <updaterate>100.0</updaterate>
+            <contact>
+              <collision>ur5/wrist_3_link_fixed_joint_lump__gripper_base_link_fixed_joint_lump__/bumper_gripper_link_collision_5</collision>
+            </contact>
+                <plugin name="gazebo_ros_bumper_controller" filename="libgazebo_ros_bumper.so">
+                    <bumperTopicName>bumper_gripper_states</bumperTopicName>
+                    <frameName>world</frameName>
+                </plugin>
+          </sensor>
+        </gazebo>
+      <!-- #############################bumper_test###############################-->
         <gazebo reference="${prefix}gripper_finger2_finger_tip_link">
             <implicitSpringDamper>1</implicitSpringDamper>

Commit message: update gripper code

File: robotiq_85_description/urdf/robotiq_85_gripper.urdf.xacro (robot description, xacro)
@@ -308,10 +308,10 @@
               </material>
           </visual> -->
-          <collision name="${prefix}gripper_base_link_fixed_joint_lump__${prefix}/bumper_gripper_link">
+          <!-- <collision name="${prefix}gripper_base_link_fixed_joint_lump__${prefix}/bumper_gripper_link">
               <origin rpy="0 0 0" xyz="0.168 0 0"/>
               <geometry>
                   <box size="0.01 0.13 0.11"/>
               </geometry>
-          </collision>
+          </collision> -->
         </link>
         <joint name="${prefix}bumper_gripper_joint" type="fixed">
@@ -348,10 +348,14 @@
               <gripper_link>${prefix}gripper_finger1_finger_tip_link</gripper_link>
               <gripper_link>${prefix}gripper_finger2_finger_tip_link</gripper_link>
+              <gripper_link>${prefix}gripper_finger2_knuckle_link</gripper_link>
+              <gripper_link>${prefix}gripper_finger1_knuckle_link</gripper_link>
+              <gripper_link>${prefix}gripper_finger1_inner_knuckle_link</gripper_link>
+              <gripper_link>${prefix}gripper_finger2_inner_knuckle_link</gripper_link>
             </arm>
 	    <forces_angle_tolerance>100</forces_angle_tolerance>
-	    <update_rate>8</update_rate>
+	    <update_rate>4</update_rate>
 	    <grip_count_threshold>1</grip_count_threshold>
 	    <max_grip_count>2</max_grip_count>
-	    <release_tolerance>0.005</release_tolerance>
+	    <release_tolerance>0.05</release_tolerance>
 	    <disable_collisions_on_attach>true</disable_collisions_on_attach>
 	    <contact_topic>__default_topic__</contact_topic>
